File: piccolo.kicad_sch (KiCad schematic)
At the start: 44 parts, among them J0 CON_PICO_40W, J1 USB_C_Receptacle_USB2.0, J2 Debug, Q1 DMG1012T, SW1 BOOTSEL, U1 RP2040, U2 ME6217C33M5, U3 W25Q16JVUXIQ, X1 SIT1602AI-22-33E-12.000000

Commit message: value-engineered for jlcpcb
Parts:
- removed R2: 100k, Resistor_SMD:R_0402_1005Metric, symbol Device:R_Small
- removed SW1: BOOTSEL, Button_Switch_SMD:SW_Push_1P1T_NO_Vertical_Wuerth_434133025816, symbol Switch:SW_Push
- removed U2: ME6217C33M5, Package_TO_SOT_SMD:SOT-23-5, symbol agausmann:ME6217C33M5
- added SW2: TS-1187A-B-A-B, SW_TS-1187A-B-A-B, symbol TS-1187A-B-A-B:TS-1187A-B-A-B
- added U4: AMS1117-3.3, Package_TO_SOT_SMD:SOT-223-3_TabPin2, symbol Regulator_Linear:AMS1117-3.3
- added Y1: 12MHz, Crystal:Crystal_SMD_3225-4Pin_3.2x2.5mm, symbol Device:Crystal_GND24
- C10: renamed from C8; footprint Capacitor_SMD:C_0201_0603Metric -> Capacitor_SMD:C_0402_1005Metric; LCSC C160831 -> C1525
- C11: renamed from C10; footprint Capacitor_SMD:C_0201_0603Metric -> Capacitor_SMD:C_0402_1005Metric; LCSC C160831 -> C1525
- C13: renamed from C9; footprint Capacitor_SMD:C_0201_0603Metric -> Capacitor_SMD:C_0402_1005Metric; LCSC C160831 -> C1525
- C15: renamed from C11; footprint Capacitor_SMD:C_0201_0603Metric -> Capacitor_SMD:C_0402_1005Metric; LCSC C160831 -> C1525
- C17: renamed from C16; footprint Capacitor_SMD:C_0201_0603Metric -> Capacitor_SMD:C_0402_1005Metric; LCSC C160831 -> C1525; now not fitted
- C2: renamed from C15; footprint Capacitor_SMD:C_0201_0603Metric -> Capacitor_SMD:C_0402_1005Metric; LCSC C160831 -> C1525
- C3: LCSC C66942 -> C1523
- C5: renamed from C4; footprint Capacitor_SMD:C_0201_0603Metric -> Capacitor_SMD:C_0402_1005Metric; LCSC C160831 -> C1525
- C7: renamed from C6; footprint Capacitor_SMD:C_0201_0603Metric -> Capacitor_SMD:C_0402_1005Metric; LCSC C160831 -> C1525
- C8: renamed from C5; footprint Capacitor_SMD:C_0201_0603Metric -> Capacitor_SMD:C_0402_1005Metric; LCSC C160831 -> C1525
- C9: renamed from C7; footprint Capacitor_SMD:C_0201_0603Metric -> Capacitor_SMD:C_0402_1005Metric; LCSC C160831 -> C1525
- U3: renamed from U1; footprint agausmann:RP2040_QFN-56-1EP_7x7mm_P0.4mm_EP3.2x3.2mm_ThermalVias -> Package_DFN_QFN:QFN-56-1EP_7x7mm_P0.4mm_EP3.2x3.2mm
- X1: footprint agausmann:SiT1602xx-2_3.2x2.5mm -> Crystal:Crystal_SMD_SeikoEpson_TSX3225-4Pin_3.2x2.5mm; now not fitted
- renumbered C18 to C1, C14 to C12, C12 to C14, C13 to C16, C1 to C4, C2 to C6, J0 to J2, J2 to J3, R4 to R1, R12 to R10, R13 to R11, R7 to R12, R9 to R13, R3 to R14, R8 to R15, R11 to R2, R16 to R3, R17 to R4, R10 to R5, R1 to R6, R5 to R7, R6 to R8, U3 to U1
Connections:
- net +3V3: now also U4.2 (VO)
- net GND: now also SW2.A, SW2.B, U4.1 (GND), Y1.2, Y1.4
- net VSYS: now also U4.3 (VI)
- net XIN: now also Y1.1
- net at R2.2: now also SW2.C, SW2.D
- net XOUT: now reaches U3.21 (XOUT)
- net XOUT: now also Y1.3
- no-connect marks 4 -> 3
Other:
- moved on the sheet: C4, D1
